Commit message: testing

File: src/lab2/urdf/three_revolute.urdf (robot description, URDF)
Before this commit: robot three_revolute, 5 links, 4 joints
Links:
- link link1: geometry visual cylinder length=0.3 radius=0.05

Commit message: testing

File: src/lab2/urdf/three_revolute.urdf (robot description, URDF)
Before this commit: robot three_revolute, 5 links, 4 joints
Links:
- link link1: geometry visual cylinder length=0.1 radius=0.05
