Commit message: Frist full wAM Model

File: src/finalProject/urdf/bt7R copy.urdf (robot description, URDF)
Before this commit: robot bt7R, 9 links, 8 joints
Links:
- removed link link5
- removed link link6
- removed link link7
- link link2: geometry 
- link link3: geometry visual sphere radius=0.05; visual sphere radius=0.05
- link link4: geometry visual cylinder length=0.55 radius=0.05
Joints:
- removed joint joint5
- removed joint joint6
- removed joint joint7
- joint map_to_base: origin xyz=0 0 0.2 rpy=0 0 0 -> xyz=0 0 0 rpy=0 0 0

File: src/lab3/urdf/puma.urdf (robot description, URDF)
Before this commit: robot puma, 8 links, 7 joints
Joints:
- joint joint1: limit (none) -> lower=-1.57 upper=1.57 effort=10.0 velocity=1.0; type continuous -> revolute
