Commit message: WAM arm with correct zero position

File: src/finalProject/urdf/bt7R.urdf (robot description, URDF)
Before this commit: robot bt7R, 9 links, 8 joints
Links:
- added link link8; visual cylinder length=0.0 radius=0.00
- link base_link: geometry 
Joints:
- added joint joint8: type fixed, parent link7, child link8, origin xyz=0 0 0.06 rpy=0 0 0, axis 0 0 1
- joint joint5: origin xyz=0 0 0.275 rpy=0 0 0 -> xyz=0 0 0.3 rpy=0 0 0
- joint map_to_base: origin xyz=0 0 0.2 rpy=0 0 0 -> xyz=0 0 0 rpy=0 0 0
